File: scm/4-Phase-BLDC-Controller.sch (KiCad schematic (older format))
At the start: 9 parts

Commit message: added BEMF feedback to schematic
Parts:
- added C? (x4): C, symbol Device:C
- added R? (x12): R, symbol Device:R
Connections:
- net PhaseA: now reaches Q?.3 (S)
- net PhaseA: now also Q?.2 (D), R?.1
- net PhaseB: now reaches Q?.3 (S)
- net PhaseB: now also Q?.2 (D), R?.1
- net PhaseC: now reaches Q?.3 (S)
- net PhaseC: now also Q?.2 (D), R?.1
- net PhaseD: now reaches Q?.3 (S)
- net PhaseD: now also Q?.2 (D), R?.1
- new net: R?.1, R?.2, R?.2 (x4)
- new net ADC-A: C?.1, R?.1
- new net ADC-B: C?.1, R?.1
- new net ADC-C: C?.1, R?.1
- new net ADC-D: C?.1, R?.1
- new net GND: C?.2, C?.2, C?.2, C?.2, R?.2, R?.2, R?.2, R?.2
Other:
- moved on the sheet: Q?
